File: PM/PM.kicad_sch (KiCad schematic)
At the start: 11 parts, among them J1 TP4056, SW1 SW_Push

Commit message: Master-Slave updated to final state for demonstration
Parts:
- added C1: 100nF, symbol Device:C_Small
- added R1: 1K, symbol Device:R
Connections:
- net GND: now also C1.1
- net Left Input: now also R1.2; no longer RV1.1
- new net: 1. (TXD/D1/GPIO43), four. (BLK)
- new net: C1.2, R1.1, RV1.1
- new net: 1. (TXD/D1/GPIO43), Two. (GND)
Changed lines of the file:
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@@
+	)
+	(junction
+		(at 50.8 46.355)
+		(diameter 0)
+		(color 0 0 0 0)
 	)
 	(junction
@@
 	)
 	(junction
+		(at 40.64 71.12)
+		(diameter 0)
+		(color 0 0 0 0)
+	)
+	(junction
 		(at 186.69 153.67)
 		(diameter 0)
@@
 	(wire
 		(pts
-			(xy 68.58 66.04) (xy 57.15 66.04)
-		)
-		(stroke
-			(width 0)
-			(type default)
-		)
-	)
-	(wire
-		(pts
 			(xy 53.34 73.66) (xy 53.34 78.74)
 		)
@@
 	(wire
 		(pts
+			(xy 50.8 46.355) (xy 54.61 46.355)
+		)
+		(stroke
+			(width 0)
+			(type default)
+		)
+	)
+	(wire
+		(pts
 			(xy 186.69 153.67) (xy 186.69 156.21)
 		)
@@
 	(wire
 		(pts
+			(xy 68.58 66.04) (xy 61.595 66.04)
+		)
+		(stroke
+			(width 0)
+			(type default)
+		)
+	)
+	(wire
+		(pts
 			(xy 190.5 133.35) (xy 193.04 133.35)
 		)
@@
 	(wire
 		(pts
+			(xy 36.195 71.12) (xy 40.64 71.12)
+		)
+		(stroke
+			(width 0)
+			(type default)
+		)
+	)
+	(wire
+		(pts
 			(xy 46.99 64.77) (xy 50.8 64.77)
 		)
@@
 	(wire
 		(pts
+			(xy 66.675 50.165) (xy 66.675 46.355)
+		)
+		(stroke
+			(width 0)
+			(type default)
+		)
+	)
+	(wire
+		(pts
 			(xy 198.12 106.68) (xy 198.12 110.49)
 		)
@@
 	(wire
 		(pts
-			(xy 57.15 54.61) (xy 50.8 54.61)
-		)
-		(stroke
-			(width 0)
-			(type default)
-		)
-	)
-	(wire
-		(pts
 			(xy 229.87 119.38) (xy 229.87 129.54)
 		)
@@
 	(wire
 		(pts
+			(xy 61.595 66.04) (xy 61.595 50.165)
+		)
+		(stroke
+			(width 0)
+			(type default)
+		)
+	)
+	(wire
+		(pts
 			(xy 195.58 115.57) (xy 190.5 115.57)
 		)
@@
 	(wire
 		(pts
+			(xy 36.195 46.355) (xy 36.195 71.12)
+		)
+		(stroke
+			(width 0)
+			(type default)
+		)
+	)
+	(wire
+		(pts
 			(xy 213.36 120.65) (xy 215.9 120.65)
 		)
@@
 	(wire
 		(pts
+			(xy 66.675 46.355) (xy 62.23 46.355)
+		)
+		(stroke
+			(width 0)
+			(type default)
+		)
+	)
+	(wire
+		(pts
 			(xy 172.72 55.88) (xy 163.83 55.88)
 		)
@@
 	(wire
 		(pts
-			(xy 50.8 54.61) (xy 50.8 55.88)
+			(xy 50.8 46.355) (xy 50.8 55.88)
 		)
 		(stroke
@@
 	(wire
 		(pts
+			(xy 41.91 46.355) (xy 36.195 46.355)
+		)
+		(stroke
+			(width 0)
+			(type default)
+		)
+	)
+	(wire
+		(pts
 			(xy 54.61 59.69) (xy 54.61 72.39)
 		)
@@
 	(wire
 		(pts
+			(xy 46.99 46.355) (xy 50.8 46.355)
+		)
+		(stroke
+			(width 0)
+			(type default)
+		)
+	)
+	(wire
+		(pts
 			(xy 46.99 73.66) (xy 53.34 73.66)
 		)
@@
 	(wire
 		(pts
+			(xy 61.595 50.165) (xy 66.675 50.165)
+		)
+		(stroke
+			(width 0)
+			(type default)
+		)
+	)
+	(wire
+		(pts
 			(xy 186.69 143.51) (xy 186.69 140.97)
-		)
-		(stroke
-			(width 0)
-			(type default)
-		)
-	)
-	(wire
-		(pts
-			(xy 57.15 66.04) (xy 57.15 54.61)
 		)
 		(stroke
@@
 	(label "GND"
 		(at 224.79 99.06 0)
-		(effects
-			(font
-				(size 1.27 1.27)
-			)
-			(justify left bottom)
-		)
-	)
-	(label "Left Input"
-		(at 52.07 54.61 0)
 		(effects
 			(font
@@
 				(path "/556d6556-7f55-4640-8331-d492643822a3"
 					(reference "four")
+					(unit 1)
+				)
+			)
+		)
+	)
+	(symbol
+		(lib_id "Device:C_Small")
+		(at 44.45 46.355 90)
+		(unit 1)
+		(body_style 1)
+		(exclude_from_sim no)
+		(in_bom yes)
+		(on_board yes)
+		(in_pos_files yes)
+		(dnp no)
+		(fields_autoplaced yes)
+		(property "Reference" "C1"
+			(at 44.4563 39.37 90)
+			(show_name no)
+			(do_not_autoplace no)
+			(effects
+				(font
+					(size 1.27 1.27)
+				)
+			)
+		)
+		(property "Value" "100nF"
+			(at 44.4563 41.91 90)
+			(show_name no)
+			(do_not_autoplace no)
+			(effects
+				(font
+					(size 1.27 1.27)
+				)
+			)
+		)
+		(property "Footprint" ""
+			(at 44.45 46.355 0)
+			(hide yes)
+			(show_name no)
+			(do_not_autoplace no)
+			(effects
+				(font
+					(size 1.27 1.27)
+				)
+			)
+		)
+		(property "Datasheet" ""
+			(at 44.45 46.355 0)
+			(hide yes)
+			(show_name no)
+			(do_not_autoplace no)
+			(effects
+				(font
+					(size 1.27 1.27)
+				)
+			)
+		)
+		(property "Description" "Unpolarized capacitor, small symbol"
+			(at 44.45 46.355 0)
+			(hide yes)
+			(show_name no)
+			(do_not_autoplace no)
+			(effects
+				(font
+					(size 1.27 1.27)
+				)
+			)
+		)
+		(pin "2"
+		)
+		(pin "1"
+		)
+		(instances
+			(project "PM"
+				(path "/556d6556-7f55-4640-8331-d492643822a3"
+					(reference "C1")
 					(unit 1)
 				)
@@
 					(unit 1)
 				)
+			)
+		)
+	)
+	(symbol
+		(lib_id "Device:R")
+		(at 58.42 46.355 90)
+		(unit 1)
+		(body_style 1)
+		(exclude_from_sim no)
+		(in_bom yes)
+		(on_board yes)
+		(in_pos_files yes)
+		(dnp no)
+		(fields_autoplaced yes)
+		(property "Reference" "R1"
+			(at 58.42 40.64 90)
+			(show_name no)
+			(do_not_autoplace no)
+			(effects
+				(font
+					(size 1.27 1.27)
+				)
+			)
+		)
+		(property "Value" "1K"
+			(at 58.42 43.18 90)
+			(show_name no)
+			(do_not_autoplace no)
+			(effects
+				(font
+					(size 1.27 1.27)
+				)
+			)
+		)
+		(property "Footprint" ""
+			(at 58.42 48.133 90)
+			(hide yes)
+			(show_name no)
+			(do_not_autoplace no)
+			(effects
+				(font
+					(size 1.27 1.27)
+				)
+			)
+		)
+		(property "Datasheet" ""
+			(at 58.42 46.355 0)
+			(hide yes)
+			(show_name no)
+			(do_not_autoplace no)
+			(effects
+				(font
+					(size 1.27 1.27)
+				)
+			)
+		)
+		(property "Description" "Resistor"
+			(at 58.42 46.355 0)
+			(hide yes)
+			(show_name no)
+			(do_not_autoplace no)
+			(effects
+				(font
+					(size 1.27 1.27)
+				)
+			)
+		)
+		(pin "2"
+		)
+		(pin "1"
+		)
+		(instances
+			(project "PM"
+				(path "/556d6556-7f55-4640-8331-d492643822a3"
+					(reference "R1")
+					(unit 1)
+				)
